File: _autosave-WN17.kicad_pcb (KiCad board)
At the start: 2 copper layers, 41 x 46 mm, 15 parts, among them J1 Conn_01x02_Pin, U1 AS5600, U2 DRV8434APWPR, U3 STM32L476RGTx, U4 ESP-12F, U5 AMS1117

Commit message: Ordered coils
Parts:
- moved U5 6.59 mm to (107.2, 78.0), turned to 0 degrees
- moved C7 6.47 mm to (98.5, 78.0)
- moved C5 1.10 mm to (125.2, 92.5)
- moved R1 0.98 mm to (124.3, 89.4), turned to 90 degrees
- moved C6 0.95 mm to (108.9, 88.7)
- moved C3 0.95 mm to (125.3, 94.5)
- moved C4 0.87 mm to (109.8, 91.6), turned to 90 degrees
- moved U4 0.70 mm to (113.0, 59.8)
- moved C2 0.66 mm to (108.8, 94.5)
- moved C1 0.20 mm to (104.1, 84.8)
Connections:
- Coils1 pad 1: unconnected-(Coils1-Pin_1-Pad1) -> DRV-BOUT1
- Coils1 pad 2: unconnected-(Coils1-Pin_2-Pad2) -> DRV-BOUT2
- Coils1 pad 3: unconnected-(Coils1-Pin_3-Pad3) -> DRV-AOUT2
- Coils1 pad 4: unconnected-(Coils1-Pin_4-Pad4) -> DRV-AOUT1
- J1 pad 1: Net-(J1-Pin_1) -> VDD
- U5 pad 3: Net-(J1-Pin_1) -> VDD
