File: PowerSupply&Connector.kicad_sch (KiCad schematic)
At the start: 3 parts, among them J1 Conn_01x02_Pin, U5 AMS1117

Commit message: Ordered coils
Parts:
- added C7: C_Polarized, Capacitor_THT:CP_Radial_D5.0mm_P2.50mm, symbol Device:C_Polarized
Connections:
- net GND: now reaches U5.1 (ADJ)
- net GND: now also J1.2 (Pin_2), C7.2
- net +3.3V: now reaches U5.2 (VO)
- net +3.3V: now also C7.1
- net VDD: now reaches U5.3 (VI)
- net VDD: now also J1.1 (Pin_1)
- net coil-B+: now reaches Coils1.1 (Pin_1)
- net coil-B-: now reaches Coils1.2 (Pin_2)
- net coil-A+: now reaches Coils1.3 (Pin_3)
- net coil-A-: now reaches Coils1.4 (Pin_4)
Other:
- moved on the sheet: U5

Commit message: Changes
Parts:
- C7: value C_Polarized -> 22uF/50V
Other:
- moved on the sheet: C7, J1, U5

Commit message: uPDATE
Parts:
- added R3: 0.01R, Resistor_SMD:R_1206_3216Metric_Pad1.30x1.75mm_HandSolder, symbol Device:R
- added U6: MCP6C02T-020E/CHY, SOT-23-6_CHY_MCH, symbol MCP6c02:MCP6C02T-020E_CHY
- J1: value Conn_01x02_Pin -> PowerIn
Connections:
- net +3.3V: now also U6.6 (VDD)
- net GND: now also U6.2 (VSS), U6.5 (VREF)
- net VDD: now also R3.2, U6.4 (VIM); no longer J1.1 (Pin_1)
- new net: J1.1 (Pin_1), R3.1, U6.3 (VIP)
- new net MCP6C02_VOUT: U6.1 (VOUT)
Other:
- note added: "P = 200 mW"
- note added: "R = V/I = 0.1V * 2 A = 0.2 Ohms"
- moved on the sheet: C7, J1, U5
